File: tfln_modulator.kicad_pcb (KiCad board)
At the start: 2 copper layers, 90 x 50 mm, 4 parts, among them J1 RF_IN, J2 RF_OUT, U1 TFLN_MODULATOR, U2 SPI_CTRL

Commit message: Added files to main
Parts:
- removed J1: RF_IN, Connector_Coaxial:SMA_Amphenol_132289_EdgeMount
- removed J2: RF_OUT, Connector_Coaxial:SMA_Amphenol_132289_EdgeMount
- removed U1: TFLN_MODULATOR, OptoDevice:Lightpipe_Bivar_RLP3-2300
- removed U2: SPI_CTRL, Package_SO:SOIC-8_3.9x4.9mm_P1.27mm
Routing:
- net RF_OUT: track 22.0 -> 0.00 mm
- net RF_IN: track 22.0 -> 0.00 mm
- net BIAS_CTRL: track 22.0 -> 0.00 mm
- added copper zone on In2.Cu, net +3V3
- added copper zone on In1.Cu, net GND
Other:
- board size 90 x 50 mm -> 50 x 40 mm
- copper layers 2 -> 4
- rule pad_to_mask_clearance: 0 -> 0.05
- board text added: "TFLN Modulator"
- board text removed: "LightRails AI"
- board text removed: "TFLN Photonic Modulator"
